File: electronics_and_firmware/OSSG_v0p4-2S/OSSG_v0p4.kicad_pcb (KiCad board)
At the start: 4 copper layers, 85 x 9 mm, 82 parts, among them J1 Conn_01x05_Male, J2 USB_B_Micro, Q1 2SC4617R BR, Q2 2SC4617R BR, Q3 PMZ290UNE2YL, Q4 EMF20B02V, SW1 SW_SPST, SW2 Power, U1 SPH0645LMH, U2 ESP32-PICO-D4, U3 CH9102F, U4 XC61CC3002MR, U5 MP2615CGQ-Z, U6 H7650-50PR, U7 NCP167BMX330TBG

Commit message: generated stuff
Routing:
- net BATT2-: track 442.0 -> 440.1 mm
- net Net-(R9-Pad2): track 0.00 -> 0.95 mm
- net Net-(R8-Pad2): track 0.00 -> 0.95 mm
